File: tornblue/pcb/tornblue_right.sch (KiCad schematic (older format))
At the start: 80 parts, among them J1 BATT, J2 SWD, J3 BREAKOUT, J4 USB C - USB2.0, J5 BATT_PIN, Q1 AO3401A, Q2 AO3401A, SW1 SW_Push, SW10 SW_Push, SW11 SW_Push, SW12 SW_Push, SW13 SW_Push, SW14 SW_Push, SW15 SW_Push, SW16 SW_Push, SW17 SW_Push, SW18 SW_Push, SW19 EC11, SW2 SW_Push, SW20 SW_Push, SW21 SW_Push, SW22 EC11, SW23 RESET, SW24 SW_SPST, SW3 SW_Push, SW4 SW_Push, SW5 SW_Push, SW6 SW_Push, SW7 SW_Push, SW8 SW_Push, SW9 SW_Push, U1 XC6220, U2 TP4056, U3 nRF52840_holyiot_18010, U4 SRV05-4

Commit message: Add right schematic
Parts:
- removed C1, C2, C3, C4: 10uF, Diode_SMD:D_0805_2012Metric, symbol Device:C_Small
- removed D1, D10, D11, D2, D3, D4, D5, D6, D7, D8, D9: BAV70_Small, Package_TO_SOT_SMD:SOT-23, symbol kicad-keyboard-parts:BAV70_Small
- removed D12, D13, D14, D15, D16, D17: WS2812B, LED_SMD:LED_WS2812B_PLCC4_5.0x5.0mm_P3.2mm, symbol LED:WS2812B
- removed D23: B5819W, Diode_SMD:D_SOD-123, symbol Device:D_Schottky_Small
- removed D25: BLUE, LED_SMD:LED_0805_2012Metric, symbol Device:LED_Small
- removed D26, D27, D28: GREEN, LED_SMD:LED_0805_2012Metric, symbol Device:LED_Small
- removed F1: 750mA, Fuse:Fuse_1206_3216Metric, symbol Device:Fuse
- removed H1, H2, H3, H4: MountingHole, MountingHole:MountingHole_3.2mm_M3_DIN965_Pad, symbol Mechanical:MountingHole
- removed H5, H6: MountingHole, tornblue:MountingHole_3.2mm_M3_DIN965_Pad_Slot, symbol Mechanical:MountingHole
- removed J1: BATT, Connector_JST:JST_PH_S2B-PH-SM4-TB_1x02-1MP_P2.00mm_Horizontal, symbol Connector_Generic:Conn_01x02
- removed J2: SWD, tornblue:SOIC_clipProgSmall, symbol Connector:Conn_01x03_Male
- removed J3: BREAKOUT, Connector_PinHeader_1.27mm:PinHeader_1x06_P1.27mm_Vertical, symbol Connector:Conn_01x06_Male
- removed J4: USB C - USB2.0, Connector_USB:USB_C_Receptacle_XKB_U262-16XN-4BVC11, symbol Connector:USB_C_Receptacle_USB2.0
- removed J5: BATT_PIN, Connector_PinHeader_2.54mm:PinHeader_1x02_P2.54mm_Vertical, symbol Connector_Generic:Conn_01x02
- removed Q1, Q2: AO3401A, Package_TO_SOT_SMD:SOT-23, symbol Transistor_FET:AO3401A
- removed R1, R4: 100k, Resistor_SMD:R_0805_2012Metric, symbol Device:R_Small
- removed R10, R9: 5.1k, Resistor_SMD:R_0805_2012Metric, symbol Device:R_Small
- removed R11, R12, R3, R8: 1k, Resistor_SMD:R_0805_2012Metric, symbol Device:R_Small
- removed R2, R7: 2M, Resistor_SMD:R_0805_2012Metric, symbol Device:R_Small
- removed R5: 10k, Resistor_SMD:R_0805_2012Metric, symbol Device:R_Small
- removed R6: 806k, Resistor_SMD:R_0805_2012Metric, symbol Device:R_Small
- removed SW1, SW10, SW11, SW12, SW13, SW14, SW15, SW16, SW17, SW18, SW2, SW20, SW21, SW3, SW4, SW5, SW6, SW7, SW8, SW9: SW_Push, tornblue:MX_PG1350_optional, symbol Switch:SW_Push
- removed SW19, SW22: EC11, tornblue:MX_PG1350_EVQWGD001_LR_optional, symbol Device:Rotary_Encoder_Switch
- removed SW23: RESET, tornblue:SW_SPST_TS24CA, symbol Switch:SW_Push
- removed SW24: SW_SPST, Button_Switch_SMD:SW_SPDT_PCM12, symbol Switch:SW_Push_SPDT
- removed U1: XC6220, Package_TO_SOT_SMD:SOT-23-5, symbol Regulator_Linear:AP2112K-3.3
- removed U2: TP4056, Package_SO:SOIC-8-1EP_3.9x4.9mm_P1.27mm_EP2.29x3mm_ThermalVias, symbol kicad-keyboard-parts:TP4056
- removed U3: nRF52840_holyiot_18010, kicad-keyboard-parts:nRF52840_holyiot_18010, symbol tornblue-rescue:nRF52840_holyiot_18010-tornblue-tornblue-rescue
- removed U4: SRV05-4, Package_TO_SOT_SMD:SOT-23-6, symbol Power_Protection:SRV05-4
- added C5, C6, C7, C8: 10uF, Diode_SMD:D_0805_2012Metric, symbol Device:C_Small
- added D18: BLUE, LED_SMD:LED_0805_2012Metric, symbol Device:LED_Small
- added D19, D20, D21, D22, D29, D30, D31, D32, D33, D34, D35: BAV70_Small, Package_TO_SOT_SMD:SOT-23, symbol kicad-keyboard-parts:BAV70_Small
- added D24: B5819W, Diode_SMD:D_SOD-123, symbol Device:D_Schottky_Small
- added D36, D37, D38, D39, D40, D41: WS2812B, LED_SMD:LED_WS2812B_PLCC4_5.0x5.0mm_P3.2mm, symbol LED:WS2812B
- added D42, D43, D44: GREEN, LED_SMD:LED_0805_2012Metric, symbol Device:LED_Small
- added F2: 750mA, Fuse:Fuse_1206_3216Metric, symbol Device:Fuse
- added H10, H7, H8, H9: MountingHole, MountingHole:MountingHole_3.2mm_M3_DIN965_Pad, symbol Mechanical:MountingHole
- added H11, H12: MountingHole, tornblue:MountingHole_3.2mm_M3_DIN965_Pad_Slot, symbol Mechanical:MountingHole
- added J10: USB C - USB2.0, Connector_USB:USB_C_Receptacle_XKB_U262-16XN-4BVC11, symbol Connector:USB_C_Receptacle_USB2.0
- added J6: BATT, Connector_JST:JST_PH_S2B-PH-SM4-TB_1x02-1MP_P2.00mm_Horizontal, symbol Connector_Generic:Conn_01x02
- added J7: BATT_PIN, Connector_PinHeader_2.54mm:PinHeader_1x02_P2.54mm_Vertical, symbol Connector_Generic:Conn_01x02
- added J8: BREAKOUT, Connector_PinHeader_1.27mm:PinHeader_1x06_P1.27mm_Vertical, symbol Connector:Conn_01x06_Male
- added J9: SWD, tornblue:SOIC_clipProgSmall, symbol Connector:Conn_01x03_Male
- added Q3, Q4: AO3401A, Package_TO_SOT_SMD:SOT-23, symbol Transistor_FET:AO3401A
- added R13, R18, R19, R20: 1k, Resistor_SMD:R_0805_2012Metric, symbol Device:R_Small
- added R14: 10k, Resistor_SMD:R_0805_2012Metric, symbol Device:R_Small
- added R15, R16: 100k, Resistor_SMD:R_0805_2012Metric, symbol Device:R_Small
- added R17, R22: 2M, Resistor_SMD:R_0805_2012Metric, symbol Device:R_Small
- added R21: 806k, Resistor_SMD:R_0805_2012Metric, symbol Device:R_Small
- added R23, R24: 5.1k, Resistor_SMD:R_0805_2012Metric, symbol Device:R_Small
- added SW25, SW26, SW27, SW29, SW30, SW31, SW32, SW33, SW34, SW35, SW36, SW37, SW38, SW39, SW40, SW41, SW42, SW43, SW46, SW47: SW_Push, tornblue:MX_PG1350_optional, symbol Switch:SW_Push
- added SW28, SW45: EC11, tornblue:MX_PG1350_EVQWGD001_LR_optional, symbol Device:Rotary_Encoder_Switch
- added SW44: SW_SPST, Button_Switch_SMD:SW_SPDT_PCM12, symbol Switch:SW_Push_SPDT
- added SW48: RESET, tornblue:SW_SPST_TS24CA, symbol Switch:SW_Push
- added U5: TP4056, Package_SO:SOIC-8-1EP_3.9x4.9mm_P1.27mm_EP2.29x3mm_ThermalVias, symbol kicad-keyboard-parts:TP4056
- added U6: XC6220, Package_TO_SOT_SMD:SOT-23-5, symbol Regulator_Linear:AP2112K-3.3
- added U7: SRV05-4, Package_TO_SOT_SMD:SOT-23-6, symbol Power_Protection:SRV05-4
- added U8: nRF52840_holyiot_18010, kicad-keyboard-parts:nRF52840_holyiot_18010, symbol tornblue-rescue:nRF52840_holyiot_18010-tornblue-tornblue-rescue
Connections:
- new net: SW48.1, U8.21 (P0.18/RESET)
- new net: J9.2 (Pin_2), U8.31 (SWDCLK)
- new net: J9.3 (Pin_3), U8.32 (SWDIO)
- new net: R21.2, R22.1, U8.6 (P0.03/AIN1-SD)
- new net: D42.1 (K), R18.1
- new net: D43.1 (K), R19.1
- new net: D44.1 (K), R20.1
- new net: J10.B5 (CC2), R24.2
- new net: J10.A5 (CC1), R23.2
- new net: D18.1 (K), R13.1
- new net: R13.2, U5.7 (CHRG)
- new net: R14.2, U5.2 (PROG)
- new net: C7.1, D24.1 (K), Q3.2 (S), R16.1, U6.1 (VIN)
- new net: R16.2, U6.3 (EN)
- new net: C8.1, SW44.2 (B), U6.5 (VOUT)
- new net: D36.2 (DOUT), D37.4 (DIN)
- new net: D37.2 (DOUT), D38.4 (DIN)
- new net: D38.2 (DOUT), D41.4 (DIN)
- new net: D40.4 (DIN), D41.2 (DOUT)
- new net: D39.4 (DIN), D40.2 (DOUT)
- new net: D22.1 (A1), SW27.2
- new net: D22.2 (A2), SW32.2
- new net: D30.2 (A2), SW38.2
- new net: D20.2 (A2), SW30.2
- new net: D35.2 (A2), SW45.S1
- new net: D30.1 (A1), SW34.2
- new net: D31.1 (A1), SW35.2
- new net: D31.2 (A2), SW39.2
- new net: D35.1 (A1), SW43.2
- new net: D21.1 (A1), SW28.S1
- new net: D34.1 (A1), SW42.2
- new net: D20.1 (A1), SW26.2
- new net: D21.2 (A2), SW31.2
- new net: D19.1 (A1), SW25.2
- new net: D19.2 (A2), SW29.2
- new net: D33.1 (A1), SW41.2
- new net: D33.2 (A2), SW46.2
- new net: D29.1 (A1), SW33.2
- new net: D29.2 (A2), SW37.2
- new net: D32.2 (A2), SW40.2
- new net: D34.2 (A2), SW47.2
- new net: D32.1 (A1), SW36.2
- new net +3.3VP: Q4.2 (S), SW44.1 (A), U8.14 (VDD_nRF)
- new net +5VP: C5.1, D18.2 (A), D24.2 (A), F2.1, Q3.1 (G), R15.1, U5.4 (VCC), U5.8 (CE), U7.5 (VP), U8.22 (VBUS)
- new net COL_R0: SW26.1, SW35.1, SW37.1, U8.13 (P0.05/AIN3)
- new net COL_R1: SW29.1, SW34.1, SW43.1, U8.12 (P0.04/AIN2)
- new net COL_R2: SW25.1, SW28.S2, SW40.1, SW42.1, U8.11 (P0.31/AIN7-SD)
- new net COL_R3: SW31.1, SW33.1, SW36.1, SW47.1, U8.15 (P0.07)
- new net COL_R4: SW32.1, SW38.1, SW39.1, SW41.1, U8.16 (P1.09)
- new net COL_R5: SW27.1, SW30.1, SW45.S2, SW46.1, U8.17 (P0.12)
- new net ENABLE_R: Q4.1 (G), R17.2, U8.28 (P1.03-SD)
- new net ENC_RA: SW28.A, SW45.A, U8.35 (P0.09/NFC1-SD)
- new net ENC_RB: SW28.B, SW45.B, U8.36 (P0.10/NFC2-SD)
- new net EXT_R_VCC: D36.1 (VDD), D37.1 (VDD), D38.1 (VDD), D39.1 (VDD), D40.1 (VDD), D41.1 (VDD), J8.6 (Pin_6), Q4.3 (D)
- new net GND1: C5.2, C6.2, C7.2, C8.2, D36.3 (VSS), D37.3 (VSS), D38.3 (VSS), D39.3 (VSS), D40.3 (VSS), D41.3 (VSS), J10.A1 (GND), J10.A12 (GND), J10.B1 (GND), J10.B12 (GND), J10.S1 (SHIELD), J6.2 (Pin_2), J7.1 (Pin_1), J8.1 (Pin_1), J9.1 (Pin_1), R14.1, R15.2, R17.1, R18.2, R19.2, R20.2, R22.2, R23.1, R24.1, SW28.C, SW45.C, SW48.2, U5.1 (TEMP), U5.3 (GND), U6.2 (GND), U7.2 (VN), U8.1 (GND), U8.25 (GND), U8.37 (GND)
- new net GPIO_RA: J8.3 (Pin_3), U8.26 (P0.22)
- new net GPIO_RB: J8.2 (Pin_2), U8.27 (P1.00)
- new net GPIO_RC: J8.4 (Pin_4), U8.20 (P0.19)
- new net GPIO_RD: J8.5 (Pin_5), U8.19 (P0.21)
- new net LED_R1: D42.2 (A), U8.8 (P0.28/AIN4-SD)
- new net LED_R2: D43.2 (A), U8.10 (P0.30/AIN6-SD)
- new net LED_R3: D44.2 (A), U8.9 (P0.29/AIN5-SD)
- new net LED_RDATA: D36.4 (DIN), U8.18 (P0.23)
- new net ROW_R0: D19.3 (K), D29.3 (K), D33.3 (K), U8.29 (P1.01-SD)
- new net ROW_R1: D20.3 (K), D30.3 (K), D34.3 (K), U8.30 (P1.02-SD)
- new net ROW_R2: D21.3 (K), D31.3 (K), D35.3 (K), U8.33 (P1.04-SD)
- new net ROW_R3: D22.3 (K), D32.3 (K), U8.34 (P1.06-SD)
- new net USB_RD+: J10.A6 (D+), J10.B6 (D+), U7.1 (IO1), U8.24 (D+)
- new net USB_RD-: J10.A7 (D-), J10.B7 (D-), U7.6 (IO4), U8.23 (D-)
- new net VBAT_R: C6.1, J6.1 (Pin_1), J7.2 (Pin_2), Q3.3 (D), R21.1, U5.5 (BAT)
- new net VBUS_R: F2.2, J10.A4 (VBUS), J10.A9 (VBUS), J10.B4 (VBUS), J10.B9 (VBUS)
Other:
- note added: "RIGHT"

Commit message: Placed components on the right side
Parts:
- renumbered SW43 to SW28, SW28 to SW43, SW46 to SW44, SW47 to SW45, SW45 to SW46, SW44 to SW47
Changed lines of the file:
@@
 P 6900 2300
 AR Path="/61BDD08B" Ref="SW?"  Part="1"
-AR Path="/61B675D2/61BDD08B" Ref="SW44"  Part="1"
-F 0 "SW44" H 6900 1975 50  0000 C CNN
+AR Path="/61B675D2/61BDD08B" Ref="SW47"  Part="1"
+F 0 "SW47" H 6900 1975 50  0000 C CNN
 F 1 "SW_SPST" H 6900 2066 50  0000 C CNN
 F 2 "Button_Switch_SMD:SW_SPDT_PCM12" H 6900 2300 50  0001 C CNN
@@
 P 5800 8350
 AR Path="/61BDD0AE" Ref="SW?"  Part="1"
-AR Path="/61B675D2/61BDD0AE" Ref="SW45"  Part="1"
-F 0 "SW45" V 5754 8580 50  0000 L CNN
+AR Path="/61B675D2/61BDD0AE" Ref="SW46"  Part="1"
+F 0 "SW46" V 5754 8580 50  0000 L CNN
 F 1 "EC11" V 5845 8580 50  0000 L CNN
 F 2 "tornblue:MX_PG1350_EVQWGD001_LR_optional" H 5650 8510 50  0001 C CNN
@@
 P 2400 8350
 AR Path="/61BDD0CA" Ref="SW?"  Part="1"
-AR Path="/61B675D2/61BDD0CA" Ref="SW28"  Part="1"
-F 0 "SW28" V 2350 7800 50  0000 L CNN
+AR Path="/61B675D2/61BDD0CA" Ref="SW43"  Part="1"
+F 0 "SW43" V 2350 7800 50  0000 L CNN
 F 1 "EC11" V 2450 7800 50  0000 L CNN
 F 2 "tornblue:MX_PG1350_EVQWGD001_LR_optional" H 2250 8510 50  0001 C CNN
@@
 P 5100 8650
 AR Path="/61BDD0E6" Ref="SW?"  Part="1"
-AR Path="/61B675D2/61BDD0E6" Ref="SW43"  Part="1"
-F 0 "SW43" H 5100 8935 50  0000 C CNN
+AR Path="/61B675D2/61BDD0E6" Ref="SW28"  Part="1"
+F 0 "SW28" H 5100 8935 50  0000 C CNN
 F 1 "SW_Push" H 5100 8844 50  0000 C CNN
 F 2 "tornblue:MX_PG1350_optional" H 5100 8850 50  0001 C CNN
@@
 P 5900 6850
 AR Path="/61BDD12C" Ref="SW?"  Part="1"
-AR Path="/61B675D2/61BDD12C" Ref="SW47"  Part="1"
-F 0 "SW47" H 5900 7135 50  0000 C CNN
+AR Path="/61B675D2/61BDD12C" Ref="SW45"  Part="1"
+F 0 "SW45" H 5900 7135 50  0000 C CNN
 F 1 "SW_Push" H 5900 7044 50  0000 C CNN
 F 2 "tornblue:MX_PG1350_optional" H 5900 7050 50  0001 C CNN
@@
 P 5900 5650
 AR Path="/61BDD164" Ref="SW?"  Part="1"
-AR Path="/61B675D2/61BDD164" Ref="SW46"  Part="1"
-F 0 "SW46" H 5900 5935 50  0000 C CNN
+AR Path="/61B675D2/61BDD164" Ref="SW44"  Part="1"
+F 0 "SW44" H 5900 5935 50  0000 C CNN
 F 1 "SW_Push" H 5900 5844 50  0000 C CNN
 F 2 "tornblue:MX_PG1350_optional" H 5900 5850 50  0001 C CNN
@@
 VBUS_R
 $Comp
-L power:GND1 #PWR?
+L power:GND1 #PWR0112
 U 1 1 623CE4CA
 P 1900 7900
-F 0 "#PWR?" H 1900 7650 50  0001 C CNN
+F 0 "#PWR0112" H 1900 7650 50  0001 C CNN
 F 1 "GND1" V 1905 7772 50  0000 R CNN
 F 2 "" H 1900 7900 50  0001 C CNN

Commit message: Fix encoder rotation
Parts:
- SW43, SW46: footprint tornblue:MX_PG1350_EVQWGD001_LR_optional -> tornblue:MX_PG1350_EVQWGD001_UD_optional
Changed lines of the file:
@@
 F 0 "SW46" V 5754 8580 50  0000 L CNN
 F 1 "EC11" V 5845 8580 50  0000 L CNN
-F 2 "tornblue:MX_PG1350_EVQWGD001_LR_optional" H 5650 8510 50  0001 C CNN
+F 2 "tornblue:MX_PG1350_EVQWGD001_UD_optional" H 5650 8510 50  0001 C CNN
 F 3 "~" H 5800 8610 50  0001 C CNN
 F 4 "-" H 5800 8350 50  0001 C CNN "LCSC"
@@
 F 0 "SW43" V 2350 7800 50  0000 L CNN
 F 1 "EC11" V 2450 7800 50  0000 L CNN
-F 2 "tornblue:MX_PG1350_EVQWGD001_LR_optional" H 2250 8510 50  0001 C CNN
+F 2 "tornblue:MX_PG1350_EVQWGD001_UD_optional" H 2250 8510 50  0001 C CNN
 F 3 "~" H 2400 8610 50  0001 C CNN
 F 4 "-" H 2400 8350 50  0001 C CNN "LCSC"

Commit message: Routing key matrix
Connections:
- net COL_R0: now also SW25.1, SW31.1; no longer SW26.1, SW35.1
- net COL_R1: now also SW26.1, SW32.1, SW38.1; no longer SW28.1, SW29.1, SW34.1
- net COL_R2: now also SW27.1, SW33.1, SW39.1, SW43.S1; no longer SW25.1, SW40.1, SW42.1, SW43.S2
- net COL_R3: now also SW28.1, SW34.1, SW40.1, SW44.1; no longer SW31.1, SW33.1, SW36.1, SW45.1
- net COL_R4: now also SW29.1, SW35.1, SW45.1; no longer SW32.1, SW38.1, SW39.1
- net COL_R5: now also SW36.1, SW42.1, SW46.S1; no longer SW27.1, SW44.1, SW46.S2
- net ENC_RA: now also SW43.B, SW46.B; no longer SW43.A, SW46.A, U8.35 (P0.09/NFC1-SD)
- net ENC_RB: now also SW43.A, SW46.A; no longer SW43.B, SW46.B, U8.36 (P0.10/NFC2-SD)
- net LED_R1: now also U8.36 (P0.10/NFC2-SD); no longer U8.8 (P0.28/AIN4-SD)
- net LED_R2: now also U8.35 (P0.09/NFC1-SD); no longer U8.10 (P0.30/AIN6-SD)
- net LED_R3: now also U8.34 (P1.06-SD); no longer U8.9 (P0.29/AIN5-SD)
- net ROW_R0: now also D22.3 (K), D35.3 (K); no longer D19.3 (K), D33.3 (K)
- net ROW_R1: now also D32.3 (K); no longer D20.3 (K)
- net ROW_R2: now also D19.3 (K), D20.3 (K), D33.3 (K); no longer D21.3 (K), D31.3 (K), D35.3 (K), U8.33 (P1.04-SD)
- net ROW_R3: now also D21.3 (K), D31.3 (K); no longer D22.3 (K), D32.3 (K), U8.34 (P1.06-SD)
- net USB_RD+: now also U7.4 (IO3); no longer U7.1 (IO1)
- net USB_RD-: now also U7.3 (IO2); no longer U7.6 (IO4)
- net at SW27.2: now also D35.2 (A2); no longer D22.1 (A1)
- net at SW32.2: now also D32.2 (A2); no longer D22.2 (A2)
- net at SW38.2: now also D19.2 (A2); no longer D30.2 (A2)
- net at SW30.2: now also D21.2 (A2); no longer D20.2 (A2)
- net at D30.1 (A1): now also SW40.2; no longer SW34.2
- net at D31.1 (A1): now also SW39.2; no longer SW35.2
- net at D31.2 (A2): now also SW34.2; no longer SW39.2
- net at D35.1 (A1): now also SW26.2; no longer SW28.2
- net at D21.1 (A1): now also SW35.2; no longer SW43.S1
- net at D20.1 (A1): now also SW45.2; no longer SW26.2
- net at SW31.2: now also D34.2 (A2); no longer D21.2 (A2)
- net at D19.1 (A1): now also SW46.S2; no longer SW25.2
- net at SW29.2: now also D22.2 (A2); no longer D19.2 (A2)
- net at D33.1 (A1): now also SW44.2; no longer SW41.2
- net at D33.2 (A2): now also SW43.S2; no longer SW44.2
- net at SW33.2: now also D30.2 (A2); no longer D29.1 (A1)
- net at SW37.2: now also D20.2 (A2); no longer D29.2 (A2)
- net at SW36.2: now also D22.1 (A1); no longer D32.1 (A1)
- new net: D29.2 (A2), SW28.2
- new net: D29.1 (A1), SW25.2
- new net: D32.1 (A1), SW41.2
Other:
- moved on the sheet: D19, D20, D21, D22, D30, D31, D32, D33, D34, D35, SW25, SW26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

Commit message: Finish layout, via placement and silk screen
Parts:
- renumbered SW30 to SW23, SW29 to SW24, SW28 to SW25, SW27 to SW26, SW26 to SW27, SW25 to SW28, SW36 to SW29, SW35 to SW30, SW34 to SW31, SW33 to SW32, SW32 to SW33, SW31 to SW34, SW42 to SW35, SW41 to SW36, SW40 to SW37, SW39 to SW38, SW38 to SW39, SW37 to SW40, SW46 to SW41, SW45 to SW42, SW44 to SW43, SW43 to SW44, SW47 to SW52, SW48 to SW53
Connections:
- net +3.3VP: now also C8.1, U6.5 (VOUT); no longer SW52.1 (A)
- net COL_R0: now also U8.20 (P0.19); no longer U8.13 (P0.05/AIN3)
- net COL_R1: now also U8.19 (P0.21); no longer U8.12 (P0.04/AIN2)
- net COL_R2: now also U8.18 (P0.23); no longer U8.11 (P0.31/AIN7-SD)
- net COL_R3: now also U8.17 (P0.12); no longer U8.15 (P0.07)
- net COL_R5: now also U8.15 (P0.07); no longer U8.17 (P0.12)
- net ENABLE_R: now also U8.13 (P0.05/AIN3); no longer U8.28 (P1.03-SD)
- net ENC_RA: now also U8.8 (P0.28/AIN4-SD)
- net ENC_RB: now also U8.7 (P0.02/AIN0-SD)
- net GPIO_RA: now also U8.10 (P0.30/AIN6-SD); no longer U8.26 (P0.22)
- net GPIO_RB: now also U8.9 (P0.29/AIN5-SD); no longer U8.27 (P1.00)
- net GPIO_RC: now also U8.11 (P0.31/AIN7-SD); no longer U8.20 (P0.19)
- net GPIO_RD: now also U8.12 (P0.04/AIN2); no longer U8.19 (P0.21)
- net LED_RDATA: now also U8.26 (P0.22); no longer U8.18 (P0.23)
- net ROW_R0: now also U8.5 (P1.15-SD); no longer U8.29 (P1.01-SD)
- net ROW_R1: now also U8.4 (P1.13-SD); no longer U8.30 (P1.02-SD)
- net ROW_R2: now also U8.3 (P1.10-SD)
- net ROW_R3: now also U8.2 (P1.11)
- net USB_RD-: now also U7.1 (IO1); no longer U7.3 (IO2)
- net VBAT_R: now also SW52.2 (B); no longer Q3.3 (D)
- new net: Q3.3 (D), SW52.1 (A)
- no-connect marks 30 -> 25
Other:
- moved on the sheet: C7, C8, D24, Q3, R15, R16, R21, R22, SW52, U6

Commit message: Fix kibot config
Command:
~/.local/bin/kicad-exports -d docs -b tornblue.kicad_pcb -e tornblue.sch -c kibot.yaml
Connections:
- no-connect marks 25 -> 30
Changed lines of the file:
@@
 	14050 3550 14300 3550
 Wire Wire Line
-	14050 3250 14300 3250
-Wire Wire Line
-	14050 3350 14300 3350
-Wire Wire Line
-	14050 3450 14300 3450
-Wire Wire Line
 	12350 3350 12650 3350
 Wire Wire Line
@@
 	13050 4150 13050 4350
 Wire Wire Line
-	14050 3150 14300 3150
-Wire Wire Line
 	14050 2950 14850 2950
 Wire Wire Line
@@
 LED_RDATA
 Wire Wire Line
-	14050 2850 14300 2850
-Wire Wire Line
 	14050 2550 14300 2550
 Wire Wire Line
@@
 Wire Wire Line
 	12350 3050 12650 3050
+NoConn ~ 14050 3450
+NoConn ~ 14050 3350
+NoConn ~ 14050 3250
+NoConn ~ 14050 3150
+NoConn ~ 14050 2850
 $EndSCHEMATC

Commit message: Add elecrow files
Parts:
- C5, C6, C7, C8, D18, D19, D20, D21, D22, D24, D29, D30, D31, D32, D33, D34, D35, D42, D43, D44, F2, J10, Q3, Q4, R13, R14, R15, R16, R17, R18, R19, R20, R21, R22, R23, R24, SW53, U5, U6, U7: Mouser (none) -> TODO
- D36, D37, D38, D39, D40, D41: LCSC - -> C2761795; Mouser (none) -> TODO
- H10, H11, H12, H7, H8, H9, J8, J9, SW23, SW24, SW25, SW26, SW27, SW28, SW29, SW30, SW31, SW32, SW33, SW34, SW35, SW36, SW37, SW38, SW39, SW40, SW41, SW42, SW43, SW44: Mouser (none) -> -
- J6: LCSC - -> C295747; Mouser (none) -> TODO
- J7: LCSC (none) -> -; Mouser (none) -> -
- SW52: LCSC (none) -> C221841; Mouser (none) -> TODO
- U8: LCSC - -> nRF52840_holyiot_18010; Mouser (none) -> TODO

Commit message: Update to kicad 6
Parts:
- C5, C6, C7, C8: Mouser TODO -> 187-CL21A106KAYNNNE
- D19, D20, D21, D22, D29, D30, D31, D32, D33, D34, D35: Mouser TODO -> 583-BAV70
- D24: Mouser TODO -> 833-B5819W-TP
- D36, D37, D38, D39, D40, D41: Mouser TODO -> 474-COM-16346
- F2: Mouser TODO -> 504-CC12H750MA-TR
- Q3, Q4: Mouser TODO -> DMP3130L
Changed lines of the file:
@@
 F 3 "https://datasheet.lcsc.com/lcsc/1912111437_BUSSMANN-CC12H750MA-TR_C328915.pdf~" H 11550 7100 50  0001 C CNN
 F 4 "C328915" H 11550 7100 50  0001 C CNN "LCSC"
-F 5 "TODO" H 11550 7100 50  0001 C CNN "Mouser"
+F 5 "504-CC12H750MA-TR" H 11550 7100 50  0001 C CNN "Mouser"
 	1    11550 7100
 	0    1    1    0
@@
 F 3 "https://datasheet.lcsc.com/lcsc/1809140216_Changjiang-Electronics-Tech--CJ-B5819W-SL_C8598.pdf" V 5850 2050 50  0001 C CNN
 F 4 "C8598" H 5850 2050 50  0001 C CNN "LCSC"
-F 5 "TODO" H 5850 2050 50  0001 C CNN "Mouser"
+F 5 "833-B5819W-TP" H 5850 2050 50  0001 C CNN "Mouser"
 	1    5850 2050
 	0    -1   -1   0
@@
 F 3 "https://datasheet.lcsc.com/lcsc/1811121310_Samsung-Electro-Mechanics-CL21A106KAYNNNE_C15850.pdf" H 6000 2800 50  0001 C CNN
 F 4 "C15850" H 6000 2800 50  0001 C CNN "LCSC"
-F 5 "TODO" H 6000 2800 50  0001 C CNN "Mouser"
+F 5 "187-CL21A106KAYNNNE" H 6000 2800 50  0001 C CNN "Mouser"
 	1    6000 2800
 	1    0    0    -1
@@
 F 3 "https://datasheet.lcsc.com/lcsc/1811121310_Samsung-Electro-Mechanics-CL21A106KAYNNNE_C15850.pdf" H 7150 2800 50  0001 C CNN
 F 4 "C15850" H 7150 2800 50  0001 C CNN "LCSC"
-F 5 "TODO" H 7150 2800 50  0001 C CNN "Mouser"
+F 5 "187-CL21A106KAYNNNE" H 7150 2800 50  0001 C CNN "Mouser"
 	1    7150 2800
 	1    0    0    -1
@@
 F 3 "http://www.aosmd.com/pdfs/datasheet/AO3401A.pdf" H 5400 2100 50  0001 L CNN
 F 4 "C15127" H 5400 2100 50  0001 C CNN "LCSC"
-F 5 "TODO" H 5400 2100 50  0001 C CNN "Mouser"
+F 5 "DMP3130L" H 5400 2100 50  0001 C CNN "Mouser"
 	1    5400 2100
 	0    -1   1    0
@@
 F 3 "https://datasheet.lcsc.com/lcsc/1811121310_Samsung-Electro-Mechanics-CL21A106KAYNNNE_C15850.pdf" H 4050 2500 50  0001 C CNN
 F 4 "C15850" H 4050 2500 50  0001 C CNN "LCSC"
-F 5 "TODO" H 4050 2500 50  0001 C CNN "Mouser"
+F 5 "187-CL21A106KAYNNNE" H 4050 2500 50  0001 C CNN "Mouser"
 	1    4050 2500
 	1    0    0    -1
@@
 F 3 "https://datasheet.lcsc.com/lcsc/1811121310_Samsung-Electro-Mechanics-CL21A106KAYNNNE_C15850.pdf" H 2750 2400 50  0001 C CNN
 F 4 "C15850" H 2750 2400 50  0001 C CNN "LCSC"
-F 5 "TODO" H 2750 2400 50  0001 C CNN "Mouser"
+F 5 "187-CL21A106KAYNNNE" H 2750 2400 50  0001 C CNN "Mouser"
 	1    2750 2400
 	1    0    0    -1
@@
 F 3 "http://www.aosmd.com/pdfs/datasheet/AO3401A.pdf" H 8900 1700 50  0001 L CNN
 F 4 "C15127" H 8900 1700 50  0001 C CNN "LCSC"
-F 5 "TODO" H 8900 1700 50  0001 C CNN "Mouser"
+F 5 "DMP3130L" H 8900 1700 50  0001 C CNN "Mouser"
 	1    8900 1700
 	0    1    1    0
@@
 F 3 "https://cdn-shop.adafruit.com/datasheets/WS2812B.pdf" H 9000 2175 50  0001 L TNN
 F 4 "C2761795" H 8900 2550 50  0001 C CNN "LCSC"
-F 5 "TODO" H 8900 2550 50  0001 C CNN "Mouser"
+F 5 "474-COM-16346" H 8900 2550 50  0001 C CNN "Mouser"
 	1    8900 2550
 	0    1    1    0
@@
 F 3 "https://cdn-shop.adafruit.com/datasheets/WS2812B.pdf" H 9000 2875 50  0001 L TNN
 F 4 "C2761795" H 8900 3250 50  0001 C CNN "LCSC"
-F 5 "TODO" H 8900 3250 50  0001 C CNN "Mouser"
+F 5 "474-COM-16346" H 8900 3250 50  0001 C CNN "Mouser"
 	1    8900 3250
 	0    1    1    0
@@
 F 3 "https://cdn-shop.adafruit.com/datasheets/WS2812B.pdf" H 9000 3575 50  0001 L TNN
 F 4 "C2761795" H 8900 3950 50  0001 C CNN "LCSC"
-F 5 "TODO" H 8900 3950 50  0001 C CNN "Mouser"
+F 5 "474-COM-16346" H 8900 3950 50  0001 C CNN "Mouser"
 	1    8900 3950
 	0    1    1    0
@@
 F 3 "https://cdn-shop.adafruit.com/datasheets/WS2812B.pdf" H 9800 3575 50  0001 L TNN
 F 4 "C2761795" H 9700 3950 50  0001 C CNN "LCSC"
-F 5 "TODO" H 9700 3950 50  0001 C CNN "Mouser"
+F 5 "474-COM-16346" H 9700 3950 50  0001 C CNN "Mouser"
 	1    9700 3950
 	0    -1   -1   0
@@
 F 3 "https://cdn-shop.adafruit.com/datasheets/WS2812B.pdf" H 9800 2875 50  0001 L TNN
 F 4 "C2761795" H 9700 3250 50  0001 C CNN "LCSC"
-F 5 "TODO" H 9700 3250 50  0001 C CNN "Mouser"
+F 5 "474-COM-16346" H 9700 3250 50  0001 C CNN "Mouser"
 	1    9700 3250
 	0    -1   -1   0
@@
 F 3 "https://cdn-shop.adafruit.com/datasheets/WS2812B.pdf" H 9800 2175 50  0001 L TNN
 F 4 "C2761795" H 9700 2550 50  0001 C CNN "LCSC"
-F 5 "TODO" H 9700 2550 50  0001 C CNN "Mouser"
+F 5 "474-COM-16346" H 9700 2550 50  0001 C CNN "Mouser"
 	1    9700 2550
 	0    -1   -1   0
@@
 F 3 "https://datasheet.lcsc.com/lcsc/1809211023_Changjiang-Electronics-Tech--CJ-BAV70_C68978.pdf" H 5500 7100 50  0001 C CNN
 F 4 "C68978" H 5500 7100 50  0001 C CNN "LCSC"
-F 5 "TODO" H 5500 7100 50  0001 C CNN "Mouser"
+F 5 "583-BAV70" H 5500 7100 50  0001 C CNN "Mouser"
 	1    5500 7100
 	1    0    0    -1
@@
 F 3 "https://datasheet.lcsc.com/lcsc/1809211023_Changjiang-Electronics-Tech--CJ-BAV70_C68978.pdf" H 4100 10150 50  0001 C CNN
 F 4 "C68978" H 4100 10150 50  0001 C CNN "LCSC"
-F 5 "TODO" H 4100 10150 50  0001 C CNN "Mouser"
+F 5 "583-BAV70" H 4100 10150 50  0001 C CNN "Mouser"
 	1    4100 10150
 	1    0    0    -1
@@
 F 3 "https://datasheet.lcsc.com/lcsc/1809211023_Changjiang-Electronics-Tech--CJ-BAV70_C68978.pdf" H 2700 5900 50  0001 C CNN
 F 4 "C68978" H 2700 5900 50  0001 C CNN "LCSC"
-F 5 "TODO" H 2700 5900 50  0001 C CNN "Mouser"
+F 5 "583-BAV70" H 2700 5900 50  0001 C CNN "Mouser"
 	1    2700 5900
 	1    0    0    -1
@@
 F 3 "https://datasheet.lcsc.com/lcsc/1809211023_Changjiang-Electronics-Tech--CJ-BAV70_C68978.pdf" H 4100 8900 50  0001 C CNN
 F 4 "C68978" H 4100 8900 50  0001 C CNN "LCSC"
-F 5 "TODO" H 4100 8900 50  0001 C CNN "Mouser"
+F 5 "583-BAV70" H 4100 8900 50  0001 C CNN "Mouser"
 	1    4100 8900
 	1    0    0    -1
@@
 F 3 "https://datasheet.lcsc.com/lcsc/1809211023_Changjiang-Electronics-Tech--CJ-BAV70_C68978.pdf" H 5500 5900 50  0001 C CNN
 F 4 "C68978" H 5500 5900 50  0001 C CNN "LCSC"
-F 5 "TODO" H 5500 5900 50  0001 C CNN "Mouser"
+F 5 "583-BAV70" H 5500 5900 50  0001 C CNN "Mouser"
 	1    5500 5900
 	1    0    0    -1
@@
 F 3 "https://datasheet.lcsc.com/lcsc/1809211023_Changjiang-Electronics-Tech--CJ-BAV70_C68978.pdf" H 2700 8900 50  0001 C CNN
 F 4 "C68978" H 2700 8900 50  0001 C CNN "LCSC"
-F 5 "TODO" H 2700 8900 50  0001 C CNN "Mouser"
+F 5 "583-BAV70" H 2700 8900 50  0001 C CNN "Mouser"
 	1    2700 8900
 	1    0    0    -1
@@
 F 3 "https://datasheet.lcsc.com/lcsc/1809211023_Changjiang-Electronics-Tech--CJ-BAV70_C68978.pdf" H 5500 8900 50  0001 C CNN
 F 4 "C68978" H 5500 8900 50  0001 C CNN "LCSC"
-F 5 "TODO" H 5500 8900 50  0001 C CNN "Mouser"
+F 5 "583-BAV70" H 5500 8900 50  0001 C CNN "Mouser"
 	1    5500 8900
 	1    0    0    -1
@@
 F 3 "https://datasheet.lcsc.com/lcsc/1809211023_Changjiang-Electronics-Tech--CJ-BAV70_C68978.pdf" H 4100 5900 50  0001 C CNN
 F 4 "C68978" H 4100 5900 50  0001 C CNN "LCSC"
-F 5 "TODO" H 4100 5900 50  0001 C CNN "Mouser"
+F 5 "583-BAV70" H 4100 5900 50  0001 C CNN "Mouser"
 	1    4100 5900
 	1    0    0    -1
@@
 F 3 "https://datasheet.lcsc.com/lcsc/1809211023_Changjiang-Electronics-Tech--CJ-BAV70_C68978.pdf" H 2700 7100 50  0001 C CNN
 F 4 "C68978" H 2700 7100 50  0001 C CNN "LCSC"
-F 5 "TODO" H 2700 7100 50  0001 C CNN "Mouser"
+F 5 "583-BAV70" H 2700 7100 50  0001 C CNN "Mouser"
 	1    2700 7100
 	1    0    0    -1
@@
 F 3 "https://datasheet.lcsc.com/lcsc/1809211023_Changjiang-Electronics-Tech--CJ-BAV70_C68978.pdf" H 2700 10150 50  0001 C CNN
 F 4 "C68978" H 2700 10150 50  0001 C CNN "LCSC"
-F 5 "TODO" H 2700 10150 50  0001 C CNN "Mouser"
+F 5 "583-BAV70" H 2700 10150 50  0001 C CNN "Mouser"
 	1    2700 10150
 	1    0    0    -1
@@
 F 3 "https://datasheet.lcsc.com/lcsc/1809211023_Changjiang-Electronics-Tech--CJ-BAV70_C68978.pdf" H 4100 7100 50  0001 C CNN
 F 4 "C68978" H 4100 7100 50  0001 C CNN "LCSC"
-F 5 "TODO" H 4100 7100 50  0001 C CNN "Mouser"
+F 5 "583-BAV70" H 4100 7100 50  0001 C CNN "Mouser"
 	1    4100 7100
 	1    0    0    -1
