File: tornblue/pcb/tornblue.kicad_sch (KiCad schematic)
At the start: 80 parts, among them J1 BATT, J2 SWD, J3 BREAKOUT, J4 USB C - USB2.0, J5 BATT_PIN, Q1 AO3401A, Q2 AO3401A, SW1 SW_Push, SW10 SW_Push, SW11 SW_Push, SW12 SW_Push, SW13 SW_Push, SW14 SW_Push, SW15 SW_Push, SW16 SW_Push, SW17 SW_Push, SW18 SW_Push, SW19 EC11, SW2 SW_Push, SW20 SW_Push, SW21 SW_Push, SW22 EC11, SW3 SW_Push, SW4 SW_Push, SW5 SW_Push, SW50 SW_SPST, SW51 RESET, SW6 SW_Push, SW7 SW_Push, SW8 SW_Push, SW9 SW_Push, U1 XC6220, U2 TP4056, U3 nRF52840_holyiot_18010, U4 SRV05-4

Commit message: Update reset button
Parts:
- SW51: footprint tornblue:SW_SPST_TS24CA -> tornblue:SW_SPST_EVQPUC02K; LCSC C393942 -> (none)
Changed lines of the file:
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@@
     (property "Reference" "SW51" (id 0) (at 364.49 111.76 0))
     (property "Value" "RESET" (id 1) (at 364.49 109.22 0))
-    (property "Footprint" "tornblue:SW_SPST_TS24CA" (id 2) (at 364.49 101.6 0)
-      (effects (font (size 1.27 1.27)) hide)
-    )
-    (property "Datasheet" "https://datasheet.lcsc.com/lcsc/1912111437_SHOU-HAN-TS24CA_C393942.pdf" (id 3) (at 364.49 101.6 0)
-      (effects (font (size 1.27 1.27)) hide)
-    )
-    (property "LCSC" "C393942" (id 4) (at 364.49 106.68 0)
+    (property "Footprint" "tornblue:SW_SPST_EVQPUC02K" (id 2) (at 364.49 101.6 0)
+      (effects (font (size 1.27 1.27)) hide)
+    )
+    (property "Datasheet" "" (id 3) (at 364.49 101.6 0)
+      (effects (font (size 1.27 1.27)) hide)
+    )
+    (property "LCSC" "" (id 4) (at 364.49 106.68 0)
       (effects (font (size 1.27 1.27)) hide)
     )
@@
     )
     (path "/00000000-0000-0000-0000-000061115765"
-      (reference "SW51") (unit 1) (value "RESET") (footprint "tornblue:SW_SPST_TS24CA")
+      (reference "SW51") (unit 1) (value "RESET") (footprint "tornblue:SW_SPST_EVQPUC02K")
     )
     (path "/00000000-0000-0000-0000-000061b675d2/00000000-0000-0000-0000-000061bdd08b"
@@
     )
     (path "/00000000-0000-0000-0000-000061b675d2/00000000-0000-0000-0000-000061bdcf7c"
-      (reference "SW53") (unit 1) (value "RESET") (footprint "tornblue:SW_SPST_TS24CA")
+      (reference "SW53") (unit 1) (value "RESET") (footprint "tornblue:SW_SPST_EVQPUC02K")
     )
     (path "/00000000-0000-0000-0000-00006351c4cf"

Commit message: Fix 3d models without changing footrprint pads
Parts:
- D1, D10, D11, D2, D3, D4, D5, D6, D7, D8, D9, Q1, Q2: footprint Package_TO_SOT_SMD:SOT-23 -> tornblue:SOT-23
- U1: footprint Package_TO_SOT_SMD:SOT-23-5 -> tornblue:SOT-23-5
- U2: footprint Package_SO:SOIC-8-1EP_3.9x4.9mm_P1.27mm_EP2.29x3mm_ThermalVias -> tornblue:SOIC-8-1EP_3.9x4.9mm_P1.27mm_EP2.29x3mm_ThermalVias
- U3: footprint kicad-keyboard-parts:nRF52840_holyiot_18010 -> tornblue:nRF52840_holyiot_18010
- U4: footprint Package_TO_SOT_SMD:SOT-23-6 -> tornblue:SOT-23-6
