File: tornblue/pcb/tornblue.kicad_sch (KiCad schematic)
At the start: 80 parts, among them J1 BATT, J2 SWD, J3 BREAKOUT, J4 USB C - USB2.0, J5 BATT_PIN, Q1 AO3401A, Q2 AO3401A, SW1 SW_Push, SW10 SW_Push, SW11 SW_Push, SW12 SW_Push, SW13 SW_Push, SW14 SW_Push, SW15 SW_Push, SW16 SW_Push, SW17 SW_Push, SW18 SW_Push, SW19 EC11, SW2 SW_Push, SW20 SW_Push, SW21 SW_Push, SW22 EC11, SW3 SW_Push, SW4 SW_Push, SW5 SW_Push, SW50 SW_SPST, SW51 RESET, SW6 SW_Push, SW7 SW_Push, SW8 SW_Push, SW9 SW_Push, U1 XC6220, U2 TP4056, U3 nRF52840_holyiot_18010, U4 SRV05-4

Commit message: checkpoint
Parts:
- J2: symbol Connector:Conn_01x03_Male -> Connector:Conn_01x04_Male
Connections:
- net +3V3: now also J2.4 (Pin_4)
Changed lines of the file:
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@@
     (stroke (width 0) (type default) (color 0 0 0 0))
   )
-  (wire (pts (xy 374.65 78.74) (xy 373.38 78.74))
-    (stroke (width 0) (type default) (color 0 0 0 0))
-  )
   (wire (pts (xy 259.08 107.95) (xy 259.08 100.33))
     (stroke (width 0) (type default) (color 0 0 0 0))
@@
     (stroke (width 0) (type default) (color 0 0 0 0))
   )
-  (wire (pts (xy 373.38 82.55) (xy 373.38 78.74))
+  (wire (pts (xy 374.65 82.55) (xy 374.65 78.74))
     (stroke (width 0) (type default) (color 0 0 0 0))
   )
@@
     (stroke (width 0) (type default) (color 0 0 0 0))
   )
+  (wire (pts (xy 374.65 67.31) (xy 374.65 71.12))
+    (stroke (width 0) (type default) (color 0 0 0 0))
+  )
   (image (at 40.64 60.96)
     (data
@@
     (pin "1")
   )
-  (symbol (lib_id "power:GND") (at 373.38 82.55 0) (unit 1)
+  (symbol (lib_id "power:GND") (at 374.65 82.55 0) (unit 1)
     (in_bom yes) (on_board yes)
-    (property "Reference" "#PWR07" (id 0) (at 373.38 88.9 0)
+    (property "Reference" "#PWR07" (id 0) (at 374.65 88.9 0)
       (effects (font (size 1.27 1.27)) hide)
     )
-    (property "Value" "GND" (id 1) (at 373.507 86.9442 0))
-    (property "Footprint" "" (id 2) (at 373.38 82.55 0)
+    (property "Value" "GND" (id 1) (at 374.777 86.9442 0))
+    (property "Footprint" "" (id 2) (at 374.65 82.55 0)
       (effects (font (size 1.27 1.27)) hide)
     )
-    (property "Datasheet" "" (id 3) (at 373.38 82.55 0)
+    (property "Datasheet" "" (id 3) (at 374.65 82.55 0)
       (effects (font (size 1.27 1.27)) hide)
     )
@@
     (pin "2")
   )
-  (symbol (lib_id "Connector:Conn_01x03_Male") (at 379.73 76.2 180) (unit 1)
+  (symbol (lib_id "Connector:Conn_01x04_Male") (at 379.73 76.2 180) (unit 1)
     (in_bom yes) (on_board yes)
     (property "Reference" "J2" (id 0) (at 383.54 78.74 0)
@@
     (pin "2")
     (pin "3")
+    (pin "4")
   )
   (symbol (lib_id "power:PWR_FLAG") (at 311.15 179.07 0) (unit 1)
@@
     (pin "1")
   )
+  (symbol (lib_id "power:+3.3V") (at 374.65 67.31 0) (unit 1)
+    (in_bom yes) (on_board yes) (fields_autoplaced)
+    (property "Reference" "#PWR0117" (id 0) (at 374.65 71.12 0)
+      (effects (font (size 1.27 1.27)) hide)
+    )
+    (property "Value" "+3.3V" (id 1) (at 374.65 62.23 0))
+    (property "Footprint" "" (id 2) (at 374.65 67.31 0)
+      (effects (font (size 1.27 1.27)) hide)
+    )
+    (property "Datasheet" "" (id 3) (at 374.65 67.31 0)
+      (effects (font (size 1.27 1.27)) hide)
+    )
+    (pin "1")
+  )
   (sheet (at 203.2 250.19) (size 50.8 25.4) (fields_autoplaced)
     (stroke (width 0) (type solid) (color 0 0 0 0))
@@
       (reference "#PWR0116") (unit 1) (value "GND1") (footprint "")
     )
+    (path "/79ba0572-2056-43c1-be53-6ceefc2cf25a"
+      (reference "#PWR0117") (unit 1) (value "+3.3V") (footprint "")
+    )
     (path "/00000000-0000-0000-0000-000061b675d2/00000000-0000-0000-0000-000062245a7f"
       (reference "#PWR0118") (unit 1) (value "GND1") (footprint "")
@@
       (reference "#PWR0127") (unit 1) (value "GND1") (footprint "")
     )
+    (path "/00000000-0000-0000-0000-000061b675d2/f3045f67-283a-4d9e-a94e-b77e3edd84d2"
+      (reference "#PWR0128") (unit 1) (value "+3.3VP") (footprint "")
+    )
     (path "/00000000-0000-0000-0000-0000650190b6"

Commit message: Update kibot for KiCad 6 and start elcrow bom
Slightly hacky but running on osx:

DYLD_FALLBACK_LIBRARY_PATH=/Applications/KiCad/KiCad.app/Contents/Frameworks:/usr/local/opt/python\@3.8/Frameworks/Python.framework/ PYTHONPATH=/Applications/KiCad/KiCad.app/Contents/Frameworks/Python.framework/Versions/3.8/lib/python3.8/site-packages/ /usr/local/opt/python@3.8/bin/python3 ../../../KiBot/src/kibot -c kibot.yaml -d docs -e tornblue.kicad_sch
Parts:
- C1, C2, C3, C4: Mouser 187-CL21A106KAYNNNE -> (none); PartNumber (none) -> 187-CL21A106KAYNNNE
- D1, D10, D11, D2, D3, D4, D5, D6, D7, D8, D9: Mouser 583-BAV70 -> (none); PartNumber (none) -> 583-BAV70
- D12, D13, D14, D15, D16, D17: Mouser 474-COM-16346 -> (none); PartNumber (none) -> 474-COM-16346; now left out of the parts list
- D23: Mouser 833-B5819W-TP -> (none); PartNumber (none) -> 833-B5819W-TP
- D25, D26, D27, D28, J4, R1, R10, R11, R12, R2, R3, R4, R5, R6, R7, R8, R9, SW50, SW51, U1, U2, U3, U4: PartNumber (none) -> TODO
- F1: Mouser 504-CC12H750MA-TR -> (none); PartNumber (none) -> 504-CC12H750MA-TR
- H1, H2, H3, H4, H5, H6, J2, J3, J5: Mouser - -> (none); PartNumber (none) -> -
- J1: PartNumber (none) -> TODO; now left out of the parts list
- Q1, Q2: Mouser DMP3130L -> (none); PartNumber (none) -> DMP3130L
- SW1, SW10, SW11, SW12, SW13, SW14, SW15, SW16, SW17, SW18, SW19, SW2, SW20, SW21, SW22, SW3, SW4, SW5, SW6, SW7, SW8, SW9: PartNumber (none) -> -

Commit message: Elecrow BOM
Parts:
- C1, C2, C3, C4: Elecrow (none) -> 302010158; Original (none) -> N; PartNumber 187-CL21A106KAYNNNE -> CL21A106KAYNNNE
- D1, D10, D11, D2, D3, D4, D5, D6, D7, D8, D9: Original (none) -> N; PartNumber 583-BAV70 -> BAV70
- D12, D13, D14, D15, D16, D17: Original (none) -> -; PartNumber 474-COM-16346 -> -
- D23: Elecrow (none) -> 304020034; Original (none) -> N; PartNumber 833-B5819W-TP -> B5819W SL
- D25: Original (none) -> N; PartNumber TODO -> 17-21/BHC-AP1Q2/3T
- D26, D27, D28: Original (none) -> N; PartNumber TODO -> MHT170UGCT
- F1: Original (none) -> N; PartNumber 504-CC12H750MA-TR -> CC12H750MA-TR
- H1, H2, H3, H4, H5, H6, J2, J3, J5, SW1, SW10, SW11, SW12, SW13, SW14, SW15, SW16, SW17, SW18, SW19, SW2, SW20, SW21, SW22, SW3, SW4, SW5, SW6, SW7, SW8, SW9: Original (none) -> -
- J1: Original (none) -> -; PartNumber TODO -> -
- J4: Original (none) -> N; PartNumber TODO -> 918-418K2023S40001
- Q1, Q2: Original (none) -> Y; PartNumber DMP3130L -> AO3401A
- R1, R4: Elecrow (none) -> 301012150; Original (none) -> N; PartNumber TODO -> 0805W8F1003T5E
- R10, R9: Elecrow (none) -> 301012180; Original (none) -> N; PartNumber TODO -> 0805W8F5101T5E
- R11, R12, R3, R8: Elecrow (none) -> 301012189; Original (none) -> N; PartNumber TODO -> 0805W8F1001T5E
- R2, R7: Original (none) -> N; PartNumber TODO -> 0805W8F2004T5E
- R5: Elecrow (none) -> 301012152; Original (none) -> N; PartNumber TODO -> 0805W8F1002T5E
- R6: Original (none) -> N; PartNumber TODO -> 0805W8F8063T5E
- SW50: Original (none) -> Y; PartNumber TODO -> PCM12SMTR
- SW51: LCSC (none) -> C79174; Original (none) -> Y; PartNumber TODO -> EVQPUC02K
- U1: Original (none) -> Y; PartNumber TODO -> XC6220B331MR-G
- U2: Original (none) -> Y; PartNumber TODO -> TP4056-42-ESOP8
- U3: Original (none) -> Y; PartNumber TODO -> YJ-18010-nRF52840
- U4: Original (none) -> N; PartNumber TODO -> SRV05-4-P-T7
Connections:
- no-connect marks 30 -> 31
