File: tornblue/pcb/tornblue_right.kicad_sch (KiCad schematic)
At the start: 80 parts, among them J10 USB C - USB2.0, J6 BATT, J7 BATT_PIN, J8 BREAKOUT, J9 SWD, Q3 AO3401A, Q4 AO3401A, SW23 SW_Push, SW24 SW_Push, SW25 SW_Push, SW26 SW_Push, SW27 SW_Push, SW28 SW_Push, SW29 SW_Push, SW30 SW_Push, SW31 SW_Push, SW32 SW_Push, SW33 SW_Push, SW34 SW_Push, SW35 SW_Push, SW36 SW_Push, SW37 SW_Push, SW38 SW_Push, SW39 SW_Push, SW40 SW_Push, SW41 EC11, SW42 SW_Push, SW43 SW_Push, SW44 EC11, SW52 SW_SPST, SW53 RESET, U5 TP4056, U6 XC6220, U7 SRV05-4, U8 nRF52840_holyiot_18010

Commit message: Update reset button
Parts:
- SW53: footprint tornblue:SW_SPST_TS24CA -> tornblue:SW_SPST_EVQPUC02K; LCSC C393942 -> (none)
Changed lines of the file:
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@@
     (property "Reference" "SW53" (id 0) (at 367.03 113.03 0))
     (property "Value" "RESET" (id 1) (at 367.03 110.49 0))
-    (property "Footprint" "tornblue:SW_SPST_TS24CA" (id 2) (at 367.03 102.87 0)
+    (property "Footprint" "tornblue:SW_SPST_EVQPUC02K" (id 2) (at 367.03 102.87 0)
       (effects (font (size 1.27 1.27)) hide)
     )
-    (property "Datasheet" "https://datasheet.lcsc.com/lcsc/1912111437_SHOU-HAN-TS24CA_C393942.pdf" (id 3) (at 367.03 102.87 0)
+    (property "Datasheet" "" (id 3) (at 367.03 102.87 0)
       (effects (font (size 1.27 1.27)) hide)
     )
-    (property "LCSC" "C393942" (id 4) (at 367.03 107.95 0)
+    (property "LCSC" "" (id 4) (at 367.03 107.95 0)
       (effects (font (size 1.27 1.27)) hide)
     )

Commit message: Fix 3d models without changing footrprint pads
Parts:
- D19, D20, D21, D22, D29, D30, D31, D32, D33, D34, D35, Q3, Q4: footprint Package_TO_SOT_SMD:SOT-23 -> tornblue:SOT-23
- U5: footprint Package_SO:SOIC-8-1EP_3.9x4.9mm_P1.27mm_EP2.29x3mm_ThermalVias -> tornblue:SOIC-8-1EP_3.9x4.9mm_P1.27mm_EP2.29x3mm_ThermalVias
- U6: footprint Package_TO_SOT_SMD:SOT-23-5 -> tornblue:SOT-23-5
- U7: footprint Package_TO_SOT_SMD:SOT-23-6 -> tornblue:SOT-23-6
- U8: footprint kicad-keyboard-parts:nRF52840_holyiot_18010 -> tornblue:nRF52840_holyiot_18010
Changed lines of the file:
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@@
     (property "Reference" "U8" (id 0) (at 339.09 30.099 0))
     (property "Value" "nRF52840_holyiot_18010" (id 1) (at 339.09 32.4104 0))
-    (property "Footprint" "kicad-keyboard-parts:nRF52840_holyiot_18010" (id 2) (at 341.63 58.42 0)
+    (property "Footprint" "tornblue:nRF52840_holyiot_18010" (id 2) (at 341.63 58.42 0)
       (effects (font (size 1.27 1.27)) hide)
     )
@@
     (property "Reference" "U7" (id 0) (at 295.91 185.42 0))
     (property "Value" "SRV05-4" (id 1) (at 309.88 185.42 0))
-    (property "Footprint" "Package_TO_SOT_SMD:SOT-23-6" (id 2) (at 320.04 208.28 0)
+    (property "Footprint" "tornblue:SOT-23-6" (id 2) (at 320.04 208.28 0)
       (effects (font (size 1.27 1.27)) hide)
     )
@@
     (property "Reference" "U5" (id 0) (at 86.995 52.705 0))
     (property "Value" "TP4056" (id 1) (at 86.995 55.0164 0))
-    (property "Footprint" "Package_SO:SOIC-8-1EP_3.9x4.9mm_P1.27mm_EP2.29x3mm_ThermalVias" (id 2) (at 86.36 52.07 0)
+    (property "Footprint" "tornblue:SOIC-8-1EP_3.9x4.9mm_P1.27mm_EP2.29x3mm_ThermalVias" (id 2) (at 86.36 52.07 0)
       (effects (font (size 1.27 1.27)) hide)
     )
@@
     (property "Reference" "U6" (id 0) (at 170.18 49.7332 0))
     (property "Value" "XC6220" (id 1) (at 170.18 52.0446 0))
-    (property "Footprint" "Package_TO_SOT_SMD:SOT-23-5" (id 2) (at 170.18 50.165 0)
+    (property "Footprint" "tornblue:SOT-23-5" (id 2) (at 170.18 50.165 0)
       (effects (font (size 1.27 1.27)) hide)
     )
@@
     (property "Reference" "Q3" (id 0) (at 137.16 59.6646 90))
     (property "Value" "AO3401A" (id 1) (at 137.16 61.976 90))
-    (property "Footprint" "Package_TO_SOT_SMD:SOT-23" (id 2) (at 139.065 58.42 0)
+    (property "Footprint" "tornblue:SOT-23" (id 2) (at 139.065 58.42 0)
       (effects (font (size 1.27 1.27) italic) (justify left) hide)
     )
@@
     (property "Reference" "Q4" (id 0) (at 226.06 49.5046 90))
     (property "Value" "AO3401A" (id 1) (at 226.06 51.816 90))
-    (property "Footprint" "Package_TO_SOT_SMD:SOT-23" (id 2) (at 224.155 48.26 0)
+    (property "Footprint" "tornblue:SOT-23" (id 2) (at 224.155 48.26 0)
       (effects (font (size 1.27 1.27) italic) (justify left) hide)
     )
@@
     (property "Reference" "D30" (id 0) (at 139.7 174.879 0))
     (property "Value" "BAV70_Small" (id 1) (at 139.7 177.1904 0))
-    (property "Footprint" "Package_TO_SOT_SMD:SOT-23" (id 2) (at 142.24 180.34 0)
+    (property "Footprint" "tornblue:SOT-23" (id 2) (at 142.24 180.34 0)
       (effects (font (size 1.27 1.27)) hide)
     )
@@
     (property "Reference" "D31" (id 0) (at 104.14 252.349 0))
     (property "Value" "BAV70_Small" (id 1) (at 104.14 254.6604 0))
-    (property "Footprint" "Package_TO_SOT_SMD:SOT-23" (id 2) (at 106.68 257.81 0)
+    (property "Footprint" "tornblue:SOT-23" (id 2) (at 106.68 257.81 0)
       (effects (font (size 1.27 1.27)) hide)
     )
@@
     (property "Reference" "D35" (id 0) (at 68.58 144.399 0))
     (property "Value" "BAV70_Small" (id 1) (at 68.58 146.7104 0))
-    (property "Footprint" "Package_TO_SOT_SMD:SOT-23" (id 2) (at 71.12 149.86 0)
+    (property "Footprint" "tornblue:SOT-23" (id 2) (at 71.12 149.86 0)
       (effects (font (size 1.27 1.27)) hide)
     )
@@
     (property "Reference" "D20" (id 0) (at 104.14 220.599 0))
     (property "Value" "BAV70_Small" (id 1) (at 104.14 222.9104 0))
-    (property "Footprint" "Package_TO_SOT_SMD:SOT-23" (id 2) (at 106.68 226.06 0)
+    (property "Footprint" "tornblue:SOT-23" (id 2) (at 106.68 226.06 0)
       (effects (font (size 1.27 1.27)) hide)
     )
@@
     (property "Reference" "D22" (id 0) (at 139.7 144.399 0))
     (property "Value" "BAV70_Small" (id 1) (at 139.7 146.7104 0))
-    (property "Footprint" "Package_TO_SOT_SMD:SOT-23" (id 2) (at 142.24 149.86 0)
+    (property "Footprint" "tornblue:SOT-23" (id 2) (at 142.24 149.86 0)
       (effects (font (size 1.27 1.27)) hide)
     )
@@
     (property "Reference" "D19" (id 0) (at 68.58 220.599 0))
     (property "Value" "BAV70_Small" (id 1) (at 68.58 222.9104 0))
-    (property "Footprint" "Package_TO_SOT_SMD:SOT-23" (id 2) (at 71.12 226.06 0)
+    (property "Footprint" "tornblue:SOT-23" (id 2) (at 71.12 226.06 0)
       (effects (font (size 1.27 1.27)) hide)
     )
@@
     (property "Reference" "D33" (id 0) (at 139.7 220.599 0))
     (property "Value" "BAV70_Small" (id 1) (at 139.7 222.9104 0))
-    (property "Footprint" "Package_TO_SOT_SMD:SOT-23" (id 2) (at 142.24 226.06 0)
+    (property "Footprint" "tornblue:SOT-23" (id 2) (at 142.24 226.06 0)
       (effects (font (size 1.27 1.27)) hide)
     )
@@
     (property "Reference" "D29" (id 0) (at 104.14 144.399 0))
     (property "Value" "BAV70_Small" (id 1) (at 104.14 146.7104 0))
-    (property "Footprint" "Package_TO_SOT_SMD:SOT-23" (id 2) (at 106.68 149.86 0)
+    (property "Footprint" "tornblue:SOT-23" (id 2) (at 106.68 149.86 0)
       (effects (font (size 1.27 1.27)) hide)
     )
@@
     (property "Reference" "D34" (id 0) (at 68.58 174.879 0))
     (property "Value" "BAV70_Small" (id 1) (at 68.58 177.1904 0))
-    (property "Footprint" "Package_TO_SOT_SMD:SOT-23" (id 2) (at 71.12 180.34 0)
+    (property "Footprint" "tornblue:SOT-23" (id 2) (at 71.12 180.34 0)
       (effects (font (size 1.27 1.27)) hide)
     )
@@
     (property "Reference" "D21" (id 0) (at 68.58 252.349 0))
     (property "Value" "BAV70_Small" (id 1) (at 68.58 254.6604 0))
-    (property "Footprint" "Package_TO_SOT_SMD:SOT-23" (id 2) (at 71.12 257.81 0)
+    (property "Footprint" "tornblue:SOT-23" (id 2) (at 71.12 257.81 0)
       (effects (font (size 1.27 1.27)) hide)
     )
@@
     (property "Reference" "D32" (id 0) (at 104.14 174.879 0))
     (property "Value" "BAV70_Small" (id 1) (at 104.14 177.1904 0))
-    (property "Footprint" "Package_TO_SOT_SMD:SOT-23" (id 2) (at 106.68 180.34 0)
-      (effects (font (size 1.27 1.27)) hide)
-    )
+    (property "Footprint" "tornblue:SOT-23" (id 2) (at 106.68 180.34 0)
+      (effects (font (size 1.27 1.27)) hide)
+    )
