File: tornblue/pcb/tornblue_right.kicad_sch (KiCad schematic)
At the start: 80 parts, among them J10 USB C - USB2.0, J6 BATT, J7 BATT_PIN, J8 BREAKOUT, J9 SWD, Q3 AO3401A, Q4 AO3401A, SW23 SW_Push, SW24 SW_Push, SW25 SW_Push, SW26 SW_Push, SW27 SW_Push, SW28 SW_Push, SW29 SW_Push, SW30 SW_Push, SW31 SW_Push, SW32 SW_Push, SW33 SW_Push, SW34 SW_Push, SW35 SW_Push, SW36 SW_Push, SW37 SW_Push, SW38 SW_Push, SW39 SW_Push, SW40 SW_Push, SW41 EC11, SW42 SW_Push, SW43 SW_Push, SW44 EC11, SW52 SW_SPST, SW53 RESET, U5 TP4056, U6 XC6220, U7 SRV05-4, U8 nRF52840_holyiot_18010

Commit message: checkpoint
Parts:
- J9: symbol Connector:Conn_01x03_Male -> Connector:Conn_01x04_Male
Connections:
- net +3.3VP: now also J9.4 (Pin_4)
Changed lines of the file:
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@@
     (stroke (width 0) (type default) (color 0 0 0 0))
   )
-  (wire (pts (xy 375.92 83.82) (xy 375.92 80.01))
-    (stroke (width 0) (type default) (color 0 0 0 0))
-  )
   (wire (pts (xy 53.34 243.84) (xy 53.34 251.46))
     (stroke (width 0) (type default) (color 0 0 0 0))
@@
     (stroke (width 0) (type default) (color 0 0 0 0))
   )
-  (wire (pts (xy 377.19 80.01) (xy 375.92 80.01))
-    (stroke (width 0) (type default) (color 0 0 0 0))
-  )
   (wire (pts (xy 170.18 83.82) (xy 170.18 66.04))
     (stroke (width 0) (type default) (color 0 0 0 0))
@@
     (stroke (width 0) (type default) (color 0 0 0 0))
   )
+  (wire (pts (xy 377.19 69.85) (xy 377.19 72.39))
+    (stroke (width 0) (type default) (color 0 0 0 0))
+  )
   (wire (pts (xy 250.19 153.67) (xy 250.19 160.02))
     (stroke (width 0) (type default) (color 0 0 0 0))
@@
     (stroke (width 0) (type default) (color 0 0 0 0))
   )
+  (wire (pts (xy 377.19 80.01) (xy 377.19 82.55))
+    (stroke (width 0) (type default) (color 0 0 0 0))
+  )
   (wire (pts (xy 250.19 147.32) (xy 250.19 153.67))
     (stroke (width 0) (type default) (color 0 0 0 0))
@@
     (pin "2")
   )
-  (symbol (lib_id "Connector:Conn_01x03_Male") (at 382.27 77.47 180) (unit 1)
+  (symbol (lib_id "Connector:Conn_01x04_Male") (at 382.27 77.47 180) (unit 1)
     (in_bom yes) (on_board yes)
     (property "Reference" "J9" (id 0) (at 386.08 80.01 0)
@@
     (pin "2")
     (pin "3")
+    (pin "4")
   )
   (symbol (lib_id "Device:Fuse") (at 293.37 180.34 270) (unit 1)
@@
     (pin "1")
   )
-  (symbol (lib_id "power:GND1") (at 375.92 83.82 0) (unit 1)
+  (symbol (lib_id "power:GND1") (at 377.19 82.55 0) (unit 1)
     (in_bom yes) (on_board yes)
-    (property "Reference" "#PWR0124" (id 0) (at 375.92 90.17 0)
+    (property "Reference" "#PWR0124" (id 0) (at 377.19 88.9 0)
       (effects (font (size 1.27 1.27)) hide)
     )
-    (property "Value" "GND1" (id 1) (at 376.047 88.2142 0))
-    (property "Footprint" "" (id 2) (at 375.92 83.82 0)
+    (property "Value" "GND1" (id 1) (at 377.317 86.9442 0))
+    (property "Footprint" "" (id 2) (at 377.19 82.55 0)
       (effects (font (size 1.27 1.27)) hide)
     )
-    (property "Datasheet" "" (id 3) (at 375.92 83.82 0)
+    (property "Datasheet" "" (id 3) (at 377.19 82.55 0)
       (effects (font (size 1.27 1.27)) hide)
     )
@@
       (effects (font (size 1.27 1.27)) hide)
     )
+    (pin "1")
+  )
+  (symbol (lib_id "power:+3.3VP") (at 377.19 69.85 0) (unit 1)
+    (in_bom yes) (on_board yes) (fields_autoplaced)
+    (property "Reference" "#PWR0128" (id 0) (at 381 71.12 0)
+      (effects (font (size 1.27 1.27)) hide)
+    )
+    (property "Value" "+3.3VP" (id 1) (at 377.19 64.77 0))
+    (property "Footprint" "" (id 2) (at 377.19 69.85 0)
+      (effects (font (size 1.27 1.27)) hide)
+    )
+    (property "Datasheet" "" (id 3) (at 377.19 69.85 0)
+      (effects (font (size 1.27 1.27)) hide)
+    )

Commit message: Update kibot for KiCad 6 and start elcrow bom
Slightly hacky but running on osx:

DYLD_FALLBACK_LIBRARY_PATH=/Applications/KiCad/KiCad.app/Contents/Frameworks:/usr/local/opt/python\@3.8/Frameworks/Python.framework/ PYTHONPATH=/Applications/KiCad/KiCad.app/Contents/Frameworks/Python.framework/Versions/3.8/lib/python3.8/site-packages/ /usr/local/opt/python@3.8/bin/python3 ../../../KiBot/src/kibot -c kibot.yaml -d docs -e tornblue.kicad_sch
Parts:
- C5, C6, C7, C8: Mouser 187-CL21A106KAYNNNE -> (none); PartNumber (none) -> 187-CL21A106KAYNNNE
- D18, D42, D43, D44, J10, J6, R13, R14, R15, R16, R17, R18, R19, R20, R21, R22, R23, R24, SW52, SW53, U5, U6, U7, U8: PartNumber (none) -> TODO
- D19, D20, D21, D22, D29, D30, D31, D32, D33, D34, D35: Mouser 583-BAV70 -> (none); PartNumber (none) -> 583-BAV70
- D24: Mouser 833-B5819W-TP -> (none); PartNumber (none) -> 833-B5819W-TP
- D36, D37, D38, D39, D40, D41: Mouser 474-COM-16346 -> (none); PartNumber (none) -> 474-COM-16346
- F2: Mouser 504-CC12H750MA-TR -> (none); PartNumber (none) -> 504-CC12H750MA-TR
- H10, H11, H12, H7, H8, H9, J7, J8, J9: Mouser - -> (none); PartNumber (none) -> -
- Q3, Q4: Mouser DMP3130L -> (none); PartNumber (none) -> DMP3130L
- SW23, SW24, SW25, SW26, SW27, SW28, SW29, SW30, SW31, SW32, SW33, SW34, SW35, SW36, SW37, SW38, SW39, SW40, SW41, SW42, SW43, SW44: PartNumber (none) -> -

Commit message: Elecrow BOM
Parts:
- C5, C6, C7, C8: Elecrow (none) -> 302010158; Original (none) -> N; PartNumber 187-CL21A106KAYNNNE -> CL21A106KAYNNNE
- D18: Original (none) -> N; PartNumber TODO -> 17-21/BHC-AP1Q2/3T
- D19, D20, D21, D22, D29, D30, D31, D32, D33, D34, D35: Original (none) -> N; PartNumber 583-BAV70 -> BAV70
- D24: Elecrow (none) -> 304020034; Original (none) -> N; PartNumber 833-B5819W-TP -> B5819W SL
- D36, D37, D38, D39, D40, D41: Original (none) -> -; PartNumber 474-COM-16346 -> -
- D42, D43, D44: Original (none) -> N; PartNumber TODO -> MHT170UGCT
- F2: Original (none) -> N; PartNumber 504-CC12H750MA-TR -> CC12H750MA-TR
- H10, H11, H12, H7, H8, H9, J7, J8, J9, SW23, SW24, SW25, SW26, SW27, SW28, SW29, SW30, SW31, SW32, SW33, SW34, SW35, SW36, SW37, SW38, SW39, SW40, SW41, SW42, SW43, SW44: Original (none) -> -
- J10: Original (none) -> N; PartNumber TODO -> 918-418K2023S40001
- J6: Original (none) -> -; PartNumber TODO -> -
- Q3, Q4: Original (none) -> Y; PartNumber DMP3130L -> AO3401A
- R13, R18, R19, R20: Elecrow (none) -> 301012189; Original (none) -> N; PartNumber TODO -> 0805W8F1001T5E
- R14: Elecrow (none) -> 301012152; Original (none) -> N; PartNumber TODO -> 0805W8F1002T5E
- R15, R16: Elecrow (none) -> 301012150; Original (none) -> N; PartNumber TODO -> 0805W8F1003T5E
- R17, R22: Original (none) -> N; PartNumber TODO -> 0805W8F2004T5E
- R21: Original (none) -> N; PartNumber TODO -> 0805W8F8063T5E
- R23, R24: Elecrow (none) -> 301012180; Original (none) -> N; PartNumber TODO -> 0805W8F5101T5E
- SW52: Original (none) -> Y; PartNumber TODO -> PCM12SMTR
- SW53: LCSC (none) -> C79174; Original (none) -> Y; PartNumber TODO -> EVQPUC02K
- U5: Original (none) -> Y; PartNumber TODO -> TP4056-42-ESOP8
- U6: Original (none) -> Y; PartNumber TODO -> XC6220B331MR-G
- U7: Original (none) -> N; PartNumber TODO -> SRV05-4-P-T7
- U8: Original (none) -> Y; PartNumber TODO -> YJ-18010-nRF52840
